Commit message: Working version for gazebo sim

File: description/camera.xacro (robot description, xacro)
@@ -23,21 +23,20 @@
         <sensor name="camera" type="camera">
             <pose>0 0 0 0 0 0</pose>
+            <always_on>true</always_on>
             <visualize>true</visualize>
             <update_rate>10</update_rate>
+            <topic>/camera</topic>
             <camera>
-                <horizontal_fov>1.089</horizontal_fov>
-                <image>
-                    <format>R8G8B8</format>
-                    <width>640</width>
-                    <height>480</height>
-                </image>
-                <clip>
-                    <near>0.05</near>
-                    <far>8.0</far>
-                </clip>
+            <horizontal_fov>1.089</horizontal_fov>
+            <image>
+                <format>R8G8B8</format>
+                <width>640</width>
+                <height>480</height>
+            </image>
+            <clip>
+                <near>0.05</near>
+                <far>8.0</far>
+            </clip>
             </camera>
-            <plugin name="camera_controller" filename="libgazebo_ros_camera.so">
-                <frame_name>camera_link_optical</frame_name>
-            </plugin>
         </sensor>
         <material>Gazebo/Red</material>

File: description/depth_camera.xacro (robot description, xacro)
@@ -21,25 +21,22 @@
     <link name="depth_camera_link_optical"></link>
     <gazebo reference="depth_camera_link">
-        <sensor name="depth_camera" type="depth">
+        <sensor name="depth_camera" type="depth_camera">
             <pose>0 0 0 0 0 0</pose>
+            <always_on>true</always_on>
             <visualize>true</visualize>
             <update_rate>10</update_rate>
+            <topic>/depth_camera</topic>
             <camera>
-                <horizontal_fov>1.089</horizontal_fov>
-                <image>
-                    <format>B8G8R8</format>
-                    <width>640</width>
-                    <height>480</height>
-                </image>
-                <clip>
-                    <near>0.05</near>
-                    <far>8.0</far>
-                </clip>
+            <horizontal_fov>1.089</horizontal_fov>
+            <image>
+                <format>B8G8R8</format>
+                <width>640</width>
+                <height>480</height>
+            </image>
+            <clip>
+                <near>0.05</near>
+                <far>8.0</far>
+            </clip>
             </camera>
-            <plugin name="depth_camera_controller" filename="libgazebo_ros_camera.so">
-                <frame_name>camera_link_optical</frame_name>
-                <min_depth>0.1</min_depth>
-                <max_depth>100.0</max_depth>
-            </plugin>
         </sensor>
         <material>Gazebo/Red</material>

File: description/lidar.xacro (robot description, xacro)
@@ -1,53 +1,55 @@
 <?xml version="1.0"?>
 <robot xmlns:xacro="http://www.ros.org/wiki/xacro">
-    <joint name="laser_joint" type="fixed">
-        <parent link="chassis"/>
-        <child link="laser_frame"/>
-        <origin xyz="0.1 0 0.175" rpy="0 0 0"/>
-    </joint>
-    <link name="laser_frame">
-        <visual>
-            <geometry>
-                <cylinder radius="0.05" length="0.04"/>
-            </geometry>
-            <material name="red"/>
-        </visual>
-        <collision>
-            <geometry>
-                <cylinder radius="0.05" length="0.04"/>
-            </geometry>
-        </collision>
-        <xacro:inertial_cylinder mass="0.1" length="0.04" radius="0.05">
-            <origin xyz="0 0 0" rpy="0 0 0"/>
-        </xacro:inertial_cylinder>
-    </link>
-    <gazebo reference="laser_frame">
-        <sensor name="laser" type="ray">
-            <pose>0 0 0 0 0 0</pose>
-            <visualize>false</visualize>
-            <update_rate>10</update_rate>
-            <ray>
-                <scan>
-                    <horizontal>
-                        <samples>360</samples>
-                        <!--<resolution>1</resolution>-->
-                        <min_angle>-3.14</min_angle>
-                        <max_angle>3.14</max_angle>
-                    </horizontal>
-                </scan>
-                <range>
-                    <min>0.3</min>
-                    <max>12</max>
-                </range>
-            </ray>
-            <plugin name="laser_controller" filename="libgazebo_ros_ray_sensor.so">
-                <ros>
-                    <argument>~/out:=scan</argument>
-                </ros>
-                <output_type>sensor_msgs/LaserScan</output_type>
-                <frame_name>laser_frame</frame_name>
-            </plugin>
-        </sensor>
-        <material>Gazebo/Red</material>
-    </gazebo>
+  <joint name="laser_joint" type="fixed">
+    <parent link="chassis"/>
+    <child link="laser_frame"/>
+    <origin xyz="0.1 0 0.175" rpy="0 0 0"/>
+  </joint>
+  <link name="laser_frame">
+    <visual>
+      <geometry>
+        <cylinder radius="0.05" length="0.04"/>
+      </geometry>
+      <material name="red"/>
+    </visual>
+    <collision>
+      <geometry>
+        <cylinder radius="0.05" length="0.04"/>
+      </geometry>
+    </collision>
+    <xacro:inertial_cylinder mass="0.1" length="0.04" radius="0.05">
+      <origin xyz="0 0 0" rpy="0 0 0"/>
+    </xacro:inertial_cylinder>
+  </link>
+  <gazebo reference="laser_frame">
+    <sensor name="laser" type="gpu_lidar">
+      <pose>0 0 0 0 0 0</pose>
+      <topic>/lidar</topic>
+      <visualize>false</visualize>
+      <update_rate>10</update_rate>
+      <always_on>true</always_on>
+      <ray>
+        <scan>
+          <horizontal>
+            <samples>360</samples>
+            <resolution>1</resolution>
+            <min_angle>-3.14</min_angle>
+            <max_angle>3.14</max_angle>
+          </horizontal>
+          <vertical>
+            <samples>1</samples>
+            <resolution>1</resolution>
+            <min_angle>0</min_angle>
+            <max_angle>0</max_angle>
+          </vertical>
+        </scan>
+        <range>
+          <min>0.3</min>
+          <max>12.0</max>
+          <resolution>0.01</resolution>
+        </range>
+      </ray>
+    </sensor>
+    <material>Gazebo/Red</material>
+  </gazebo>
 </robot>

File: description/robot.urdf.xacro (robot description, xacro)
@@ -1,14 +1,9 @@
 <?xml version="1.0"?>
-<robot xmlns:xacro="http://www.ros.org/wiki/xacro"  name="robot">
-    <xacro:arg name="use_ros2_control" default="true"/>
-    <xacro:include filename="robot_core.xacro"/>
-    <xacro:if value="$(arg use_ros2_control)">
-        <xacro:include filename="ros2_control.xacro"/>
-    </xacro:if>
-    <xacro:unless value="$(arg use_ros2_control)">
-        <xacro:include filename="gazebo_control.xacro"/>
-    </xacro:unless>
-    <xacro:include filename="lidar.xacro"/>
-    <xacro:include filename="camera.xacro"/>
-    <xacro:include filename="depth_camera.xacro"/>
+<robot xmlns:xacro="http://www.ros.org/wiki/xacro" name="robot">
+  <xacro:arg name="use_ros2_control" default="true"/>
+  <xacro:include filename="robot_core.xacro"/>
+  <xacro:include filename="ros2_control.xacro"/>
+  <xacro:include filename="lidar.xacro"/>
+  <xacro:include filename="camera.xacro"/>
+  <xacro:include filename="depth_camera.xacro"/>
 </robot>

File: description/ros2_control.xacro (robot description, xacro)
@@ -1,29 +1,31 @@
 <?xml version="1.0"?>
 <robot xmlns:xacro="http://www.ros.org/wiki/xacro">
-    <ros2_control name="GazeboSystem" type="system">
-        <hardware>
-            <plugin>gazebo_ros2_control/GazeboSystem</plugin>
-        </hardware>
-        <joint name="left_wheel_joint">
-            <command_interface name="velocity">
-                <param name="min">-10.0</param>
-                <param name="max">10.0</param>
-            </command_interface>
-            <state_interface name="velocity"/>
-            <state_interface name="position"/>
-        </joint>
-        <joint name="right_wheel_joint">
-            <command_interface name="velocity">
-                <param name="min">-10.0</param>
-                <param name="max">10.0</param>
-            </command_interface>
-            <state_interface name="velocity"/>
-            <state_interface name="position"/>
-        </joint>
-    </ros2_control>
-    <gazebo>
-        <plugin name="gazebo_ros2_control" filename="libgazebo_ros2_control.so">
-            <parameters>$(find ar_project)/config/my_controllers.yaml</parameters>
-        </plugin>
-    </gazebo>
+  <ros2_control name="GazeboSimSystem" type="system">
+    <hardware>
+      <plugin>gz_ros2_control/GazeboSimSystem</plugin>
+    </hardware>
+    <joint name="left_wheel_joint">
+      <command_interface name="velocity">
+        <param name="min">-10.0</param>
+        <param name="max">10.0</param>
+      </command_interface>
+      <state_interface name="velocity"/>
+      <state_interface name="position"/>
+    </joint>
+    <joint name="right_wheel_joint">
+      <command_interface name="velocity">
+        <param name="min">-10.0</param>
+        <param name="max">10.0</param>
+      </command_interface>
+      <state_interface name="velocity"/>
+      <state_interface name="position"/>
+    </joint>
+  </ros2_control>
+  <gazebo>
+    <plugin
+      filename="libgz_ros2_control-system.so"
+      name="gz_ros2_control::GazeboSimROS2ControlPlugin">
+      <parameters>$(find ar_project)/config/my_controllers.yaml</parameters>
+    </plugin>
+  </gazebo>
 </robot>

Commit message: changed camera angle and nav2 params

File: description/camera.xacro (robot description, xacro)
@@ -4,5 +4,5 @@
         <parent link="chassis"/>
         <child link="camera_link"/>
-        <origin xyz="0.455 0 0.08" rpy="0 0 0"/>
+        <origin xyz="0.455 0 0.08" rpy="0 -0.35 0"/>
     </joint>
     <link name="camera_link">
@@ -36,5 +36,5 @@
             <clip>
                 <near>0.05</near>
-                <far>8.0</far>
+                <far>10.0</far>
             </clip>
             </camera>

File: description/depth_camera.xacro (robot description, xacro)
@@ -4,5 +4,5 @@
         <parent link="chassis"/>
         <child link="depth_camera_link"/>
-        <origin xyz="0.455 0 0.08" rpy="0 0 0"/>
+        <origin xyz="0.455 0 0.08" rpy="0 -0.35 0"/>
     </joint>
     <link name="depth_camera_link">
@@ -36,5 +36,5 @@
             <clip>
                 <near>0.05</near>
-                <far>8.0</far>
+                <far>10.0</far>
             </clip>
             </camera>
